Commit message: mesh: add wrist camera to SO101 model; fix wrist_roll 180° rotation
1. Add wrist camera mesh (assets/so101/assets/wrist_camera_so101_v1.stl):
   - Simple 32x32mm snap-on UVC camera with mount plate, body, and lens
   - 120 faces (lightweight, already within arm_renderer target)
   - New "camera" material (dark teal) in URDF and arm_renderer

2. Add camera visual to gripper_link in URDF:
   - Positioned at T_cam_to_gripper from cameras.yaml
   - xyz="0.01 -0.02 -0.035" rpy="3.14159 0 0" (lens faces downward)

3. Fix wrist_roll 180° rotation offset in servo_offsets.yaml:
   - The URDF wrist mesh was 180° rotated from physical reality at servo zero
   - Added urdf_offsets_deg.wrist_roll: 180.0 so FK/IK matches real arm
   - Also updated ~/.config/202602hackathon/servo_offsets.yaml (active config)

All 644 tests pass.

File: assets/so101/so101_new_calib.urdf (robot description, URDF)
Before this commit: robot so101_new_calib, 8 links, 7 joints
Links:
- link gripper_link: geometry collision mesh filename=assets/sts3215_03a_v1.stl; collision mesh filename=assets/wrist_roll_follower_so101_v1.stl
