Commit message: Replace URDF collision meshes with geometric primitives
Use box/cylinder collision primitives instead of high-detail STL meshes
in both nova5_robot.urdf and so101_new_calib.urdf.

Motivation:
- Avoids open-mesh / watertightness issues with STL geometry in FCL
- Substantially faster collision checking in MoveIt/pinocchio
- Eliminates need to carry mesh files for collision-only use

Nova5 (7 links):
  base_link  → cylinder r=75mm h=240mm
  Link1      → box 120×100×120mm (shoulder housing)
  Link2      → box 420×80×120mm (upper arm, spans ~400mm in -x)
  Link3      → box 370×70×180mm (forearm, spans ~330mm in -x, 135mm in z)
  Link4      → box 80×140×90mm (wrist-1)
  Link5      → box 80×120×75mm (wrist-2)
  Link6      → cylinder r=40mm h=45mm (end-effector flange)

SO-ARM101 (7 links, consolidated multi-part collision per link):
  base_link              → box 115×90×98mm
  shoulder_link          → box 135×55×110mm
  upper_arm_link         → box 155×60×55mm
  lower_arm_link         → box 165×70×50mm
  wrist_link             → box 48×90×75mm
  gripper_link           → box 42×45×110mm
  moving_jaw_so101_v1_link → box 30×60×60mm

Visual meshes are unchanged.

File: assets/nova5_robot.urdf (robot description, URDF)
Before this commit: robot nova5_robot, 9 links, 8 joints
Links:
- link Link1: geometry collision box size=0.120 0.100 0.120; visual mesh filename=package://dobot_description/meshes/nova5/Link1.STL
- link Link2: geometry collision box size=0.420 0.080 0.120; visual mesh filename=package://dobot_description/meshes/nova5/Link2.STL
- link Link3: geometry collision box size=0.370 0.070 0.180; visual mesh filename=package://dobot_description/meshes/nova5/Link3.STL
- link Link4: geometry collision box size=0.080 0.140 0.090; visual mesh filename=package://dobot_description/meshes/nova5/Link4.STL
- link Link5: geometry collision box size=0.080 0.120 0.075; visual mesh filename=package://dobot_description/meshes/nova5/Link5.STL
- link Link6: geometry collision cylinder length=0.045 radius=0.040; visual mesh filename=package://dobot_description/meshes/nova5/Link6.STL
- link base_link: geometry collision cylinder length=0.240 radius=0.075; visual mesh filename=package://dobot_description/meshes/nova5/base_link.STL

File: assets/so101/so101_new_calib.urdf (robot description, URDF)
Before this commit: robot so101_new_calib, 8 links, 7 joints
Links:
- link base_link: geometry collision box size=0.115 0.090 0.098; visual mesh filename=assets/base_motor_holder_so101_v1.stl
- link gripper_link: geometry collision box size=0.042 0.045 0.110; visual mesh filename=assets/sts3215_03a_v1.stl
- link lower_arm_link: geometry collision box size=0.165 0.070 0.050; visual mesh filename=assets/motor_holder_so101_wrist_v1.stl
- link moving_jaw_so101_v1_link: geometry collision box size=0.030 0.060 0.060; visual mesh filename=assets/moving_jaw_so101_v1.stl
- link shoulder_link: geometry collision box size=0.135 0.055 0.110; visual mesh filename=assets/motor_holder_so101_base_v1.stl
- link upper_arm_link: geometry collision box size=0.155 0.060 0.055; visual mesh filename=assets/sts3215_03a_v1.stl
- link wrist_link: geometry collision box size=0.048 0.090 0.075; visual mesh filename=assets/sts3215_03a_no_horn_v1.stl

Commit message: Split Link2 and Link3 collision geometry into compound primitives
Replace single conservative bounding boxes with two smaller, more accurate
collision geometries per link:
- Cylinder for arm tube (long, thin, ~330-280mm)
- Box for joint housing (bulkier, ~100mm)

Benefits:
- Link2: 32.1% volume reduction (4.0M → 2.7M mm³)
- Link3: 56.3% volume reduction (4.7M → 2.0M mm³)
- Better path planning accuracy
- Reduced false collision detections
- Geometry better matches actual arm link structure

Tested: URDF parsing, multi-collision element support verified.

File: assets/nova5_robot.urdf (robot description, URDF)
Before this commit: robot nova5_robot, 9 links, 8 joints
Links:
- link Link2: geometry collision box size=0.100 0.090 0.120; collision cylinder length=0.330 radius=0.040
- link Link3: geometry collision box size=0.100 0.080 0.120; collision cylinder length=0.280 radius=0.035
